File: Sofle_Choc/Case/PCBTop/SofleKeyboardTopPlate.kicad_pcb (KiCad board)
At the start: 2 copper layers, 143.4 x 111.8 mm, 34 parts, among them SW2 KEY_SWITCH

Commit message: Update top plate
Parts:
- removed the SW2 at (178.6, 125.1)
- added SW2: KEY_SWITCH, SofleChocTop:SW_Hole, F.Cu at (235.7, 72.9)
- added SW2: KEY_SWITCH, SofleChocTop:SW_Hole, F.Cu at (235.7, 111.0)
- added SW2: KEY_SWITCH, SofleChocTop:SW_Hole, F.Cu at (235.7, 91.9)
- added SW2: KEY_SWITCH, SofleChocTop:SW_Hole, F.Cu at (235.7, 130.0)
- added SW2: KEY_SWITCH, SofleChocTop:SW_Hole, F.Cu at (81.0, 144.4)
- added SW2: KEY_SWITCH, SofleChocTop:SW_Hole, F.Cu at (235.8, 53.8)
- moved TH6 27.2 mm to (226.2, 120.8)
- moved TH7 22.5 mm to (84.0, 130.9)
- moved TH4 19.0 mm to (226.2, 63.2)
Other:
- board size 143.4 x 111.8 mm -> 179.6 x 122.1 mm
- net class Default removed
- board text removed: "Original design by Josef Adamacik"
- board text removed: "Sofle Choc v2.1.1 by Brian Low"
- board text removed: "https://josefadamcik.github.io/SofleKeyboard/"
